File: Elektro/altimetrModul.brd (EAGLE design)
At the start: 29.2 x 13 mm, 16 parts, among them IC1 ATTINY1624-SSU, J1 SM04B-GHS-TB(LF)(SN)-

Commit message: Added Modules
Parts:
- moved JP4 36.9 mm to (7.62, 17.8)
- moved JP2 35.0 mm to (31.8, 11.4), turned to 90 degrees
Connections:
- net MISO: now also JP4.3
- net MOSI: no longer JP4.3
Routing:
- net MISO: track 10.1 -> 47.4 mm, vias 2 -> 1
- net MOSI: track 10.0 -> 38.2 mm, vias 1 -> 0
- net +3.3V: track 44.6 -> 67.8 mm, vias 3 -> 2
- net SCK: track 9.29 -> 29.1 mm
- net CS_BMP: track 11.4 -> 21.6 mm, vias 1 -> 0
- net WP: track 7.07 -> 0.00 mm
- net CS_FLASH: track 11.6 -> 17.9 mm
- net LED: track 4.23 -> 3.14 mm
- net GND: vias 0 -> 3
Other:
- board size 29.2 x 13 mm -> 35.5 x 19.4 mm

Commit message: Added names
Parts:
- removed JP2, JP4: (no value), pinhead:1X06
- added BMP_280, FLASH_: (no value), pinhead:1X06
- moved C1 6.18 mm to (18.5, 13.2), turned to 0 degrees
- moved JP3 0.89 mm to (8.51, -0.51)
Connections:
- net +3.3V: now also BMP_280.1, FLASH_.1; no longer JP2.1, JP4.1
- net CS_BMP: now also BMP_280.5; no longer JP2.5
- net CS_FLASH: now also FLASH_.2; no longer JP4.2
- net GND: now also BMP_280.2, FLASH_.4; no longer JP2.2, JP4.4
- net MISO: now also BMP_280.6, FLASH_.3; no longer JP2.6, JP4.3
- net MOSI: now also BMP_280.4, FLASH_.6; no longer JP2.4, JP4.6
- net SCK: now also BMP_280.3, FLASH_.5; no longer JP2.3, JP4.5
Routing:
- net MOSI: track 38.2 -> 32.5 mm
- net CS_BMP: track 21.6 -> 17.4 mm
- net SCK: track 29.1 -> 25.6 mm
- net MISO: track 47.4 -> 44.5 mm
- net UPDI: track 11.4 -> 12.3 mm
- net CS_FLASH: track 17.9 -> 18.5 mm
- net GND: vias 3 -> 1
Other:
- board text added: "EN"
- board text added: "Krzysztof Puzio Jakub Skrzypczak Kamil Urban"

Commit message: Gerber generated in .zip
Parts:
- moved LED1 5.08 mm to (22.5, 4.32)
- moved R1 3.81 mm to (19.6, 3.30)
- moved LED2 3.56 mm to (16.9, 4.32)
- moved JP3 1.27 mm to (9.78, -0.51)
- moved C4 0.77 mm to (5.71, 11.9)
Connections:
- removed net WP: IC1.2
Routing:
- net +3.3V: track 67.9 -> 61.3 mm
- net LED: track 3.14 -> 5.43 mm
- net MOSI: track 32.5 -> 30.6 mm
- net N$14: track 4.93 -> 6.77 mm
- net SCK: track 25.6 -> 23.9 mm
- net MISO: track 44.5 -> 43.2 mm
- net UPDI: track 12.3 -> 11.3 mm
- net GND: vias 1 -> 5
